File: template/stm32_base.kicad_sch (KiCad schematic)
At the start: 41 parts, among them J1 Network Connector, J3 STDC14 STLink connector, SW1 SW_Push, U1 LD39050PU33R, U2 STM32G474RBT6, U3 SN65HVD230, Y1 8MHz

Commit message: template: reorganize schematic for better fit
Parts:
- J3: value STDC14 STLink connector -> STDC14
Connections:
- net GND: now also SW1.2; no longer SW1.1
- net T_NRST: now also SW1.1; no longer SW1.2
Other:
- note added: "STLink Connector"
- note added: "STM32 MCU"
- note removed: "STLink"
- note removed: "STM32"
- moved on the sheet: C14, C15, C16, C17, D1, D2, H1, H2, H3, H4, J3, R2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

Commit message: template: change JLCPCB parts (capacitors & resistors)
Parts:
- C1, C10, C11, C12, C14, C17, C3, C6, C9: JLCPCB C1525 -> C1525
- C13: footprint Capacitor_SMD:C_0603_1608Metric -> Capacitor_SMD:C_0402_1005Metric; JLCPCB C19666 -> C23733
- C2, C4, C5, C8: footprint Capacitor_SMD:C_0603_1608Metric -> Capacitor_SMD:C_0402_1005Metric; JLCPCB C15849 -> C52923
- C7: footprint Capacitor_SMD:C_0603_1608Metric -> Capacitor_SMD:C_0402_1005Metric; JLCPCB C57112 -> C15195
- R2, R3: footprint Resistor_SMD:R_0603_1608Metric -> Resistor_SMD:R_0402_1005Metric; JLCPCB C22775 -> C25076
- R5, R6: footprint Resistor_SMD:R_0603_1608Metric -> Resistor_SMD:R_0402_1005Metric; JLCPCB C25804 -> C25744
- TP1: Net Label (none) -> GND
- TP2: Net Label (none) -> CAN_RX
- TP3: Net Label (none) -> +5V
- TP4: Net Label (none) -> CAN_TX
- TP5: Net Label (none) -> +3.3V
Changed lines of the file:
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@@
 			)
 		)
-		(property "JLCPCB" " C1525"
+		(property "JLCPCB" "C1525"
 			(at 93.98 40.64 0)
 			(effects
@@
 			)
 		)
+		(property "Net Label" "GND"
+			(at 180.34 85.09 0)
+			(effects
+				(font
+					(size 1.27 1.27)
+				)
+				(hide yes)
+			)
+		)
 		(pin "1"
 		)
@@
 			)
 		)
-		(property "Footprint" "Resistor_SMD:R_0603_1608Metric"
+		(property "Footprint" "Resistor_SMD:R_0402_1005Metric"
 			(at 135.382 48.26 90)
 			(effects
@@
 			)
 		)
-		(property "JLCPCB" "C25804"
+		(property "JLCPCB" "C25744"
 			(at 137.16 48.26 0)
 			(effects
@@
 			)
 		)
-		(property "Footprint" "Capacitor_SMD:C_0603_1608Metric"
+		(property "Footprint" "Capacitor_SMD:C_0402_1005Metric"
 			(at 44.1452 41.91 0)
 			(effects
@@
 			)
 		)
-		(property "JLCPCB" "C15849"
+		(property "JLCPCB" "C52923"
 			(at 43.18 38.1 0)
 			(effects
@@
 			)
 		)
-		(property "Footprint" "Capacitor_SMD:C_0603_1608Metric"
+		(property "Footprint" "Capacitor_SMD:C_0402_1005Metric"
 			(at 82.2452 44.45 0)
 			(effects
@@
 			)
 		)
-		(property "JLCPCB" "C15849"
+		(property "JLCPCB" "C52923"
 			(at 81.28 40.64 0)
 			(effects
@@
 			)
 		)
-		(property "JLCPCB" " C1525"
+		(property "JLCPCB" "C1525"
 			(at 260.35 140.97 0)
 			(effects
@@
 			)
 		)
-		(property "Footprint" "Resistor_SMD:R_0603_1608Metric"
+		(property "Footprint" "Resistor_SMD:R_0402_1005Metric"
 			(at 184.912 34.29 90)
 			(effects
@@
 			)
 		)
-		(property "JLCPCB" "C22775"
+		(property "JLCPCB" "C25076"
 			(at 186.69 34.29 0)
 			(effects
@@
 			)
 		)
-		(property "JLCPCB" " C1525"
+		(property "JLCPCB" "C1525"
 			(at 41.91 118.11 0)
 			(effects
@@
 			)
 		)
-		(property "Footprint" "Resistor_SMD:R_0603_1608Metric"
+		(property "Footprint" "Resistor_SMD:R_0402_1005Metric"
 			(at 202.692 34.29 90)
 			(effects
@@
 			)
 		)
-		(property "JLCPCB" "C22775"
+		(property "JLCPCB" "C25076"
 			(at 204.47 34.29 0)
 			(effects
@@
 			)
 		)
+		(property "Net Label" "+3.3V"
+			(at 210.82 83.82 0)
+			(effects
+				(font
+					(size 1.27 1.27)
+				)
+				(hide yes)
+			)
+		)
 		(pin "1"
 		)
@@
 			)
 		)
-		(property "Footprint" "Resistor_SMD:R_0603_1608Metric"
+		(property "Footprint" "Resistor_SMD:R_0402_1005Metric"
 			(at 104.14 160.528 90)
 			(effects
@@
 			)
 		)
-		(property "JLCPCB" "C25804"
+		(property "JLCPCB" "C25744"
 			(at 104.14 158.75 0)
 			(effects
@@
 			)
 		)
-		(property "Footprint" "Capacitor_SMD:C_0603_1608Metric"
+		(property "Footprint" "Capacitor_SMD:C_0402_1005Metric"
 			(at 144.78 141.2748 0)
 			(effects
@@
 			)
 		)
-		(property "JLCPCB" "C19666"
+		(property "JLCPCB" "C23733"
 			(at 140.97 142.24 0)
 			(effects
@@
 			)
 		)
+		(property "Net Label" "+5V"
+			(at 196.85 83.82 0)
+			(effects
+				(font
+					(size 1.27 1.27)
+				)
+				(hide yes)
+			)
+		)
 		(pin "1"
 		)
@@
 			)
 		)
-		(property "Footprint" "Capacitor_SMD:C_0603_1608Metric"
+		(property "Footprint" "Capacitor_SMD:C_0402_1005Metric"
 			(at 127 105.7148 0)
 			(effects
@@
 			)
 		)
-		(property "JLCPCB" "C15849"
+		(property "JLCPCB" "C52923"
 			(at 123.19 106.68 0)
 			(effects
@@
 			)
 		)
-		(property "JLCPCB" " C1525"
+		(property "JLCPCB" "C1525"
 			(at 140.97 116.84 0)
 			(effects
@@
 			)
 		)
-		(property "JLCPCB" " C1525"
+		(property "JLCPCB" "C1525"
 			(at 140.97 129.54 0)
 			(effects
@@
 			)
 		)
+		(property "Net Label" "CAN_TX"
+			(at 204.47 71.12 0)
+			(effects
+				(font
+					(size 1.27 1.27)
+				)
+				(hide yes)
+			)
+		)
 		(pin "1"
 		)
@@
 			)
 		)
-		(property "Footprint" "Capacitor_SMD:C_0603_1608Metric"
+		(property "Footprint" "Capacitor_SMD:C_0402_1005Metric"
 			(at 45.72 104.4448 0)
 			(effects
@@
 			)
 		)
-		(property "JLCPCB" "C15849"
+		(property "JLCPCB" "C52923"
 			(at 41.91 105.41 0)
 			(effects
@@
 			)
 		)
-		(property "JLCPCB" " C1525"
+		(property "JLCPCB" "C1525"
 			(at 31.75 38.1 0)
 			(effects
@@
 			)
 		)
-		(property "JLCPCB" " C1525"
+		(property "JLCPCB" "C1525"
 			(at 137.16 29.21 0)
 			(effects
@@
 			)
 		)
-		(property "JLCPCB" " C1525"
+		(property "JLCPCB" "C1525"
 			(at 140.97 104.14 0)
 			(effects
@@
 			)
 		)
-		(property "Footprint" "Capacitor_SMD:C_0603_1608Metric"
+		(property "Footprint" "Capacitor_SMD:C_0402_1005Metric"
 			(at 127 93.0148 0)
 			(effects
@@
 			)
 		)
-		(property "JLCPCB" "C57112"
+		(property "JLCPCB" "C15195"
 			(at 123.19 93.98 0)
 			(effects
@@
 			)
 		)
+		(property "Net Label" "CAN_RX"
+			(at 186.69 71.12 0)
+			(effects
+				(font
+					(size 1.27 1.27)
+				)
+				(hide yes)
+			)
+		)
 		(pin "1"
 		)
@@
 			)
 		)
-		(property "JLCPCB" " C1525"
+		(property "JLCPCB" "C1525"
 			(at 140.97 91.44 0)
 			(effects
