File: template/stm32_base.kicad_sch (KiCad schematic)
At the start: 41 parts, among them J1 Network Connector, J3 STDC14, SW1 SW_Push, U1 LD39050PU33R, U2 STM32G474RBT6, U3 SN65HVD230, Y1 8MHz

Commit message: template: re-reference all components
Had to re-add R1 and J2, but they were replaced where they were.
Parts:
- renumbered C9 to C10, C10 to C11, C11 to C12, C12 to C13, C13 to C14, C14 to C17, C17 to C9, J3 to J2, R6 to R1, R1 to R2, R5 to R3, R2 to R4, R3 to R5
