File: sensors-pcb/stm32_base.kicad_sch (KiCad schematic)
At the start: 41 parts, among them J1 Network Connector, J2 STDC14, SW1 SW_Push, U1 LD39050PU33R, U2 STM32G474RBT6, U3 SN65HVD230, Y1 8MHz

Commit message: sensors-pcb: adjust IMU schematic and symbol
hide no connect pins
add connect I2C I/O to STM32 with pull-up resistors
add external 42kHz clock from Exocet template
pins 15 and 16 connected to GND through solder jumper
because of conflicting datasheet info (2021 vs 2016). to be tested IRL
Parts:
- renumbered C6 to C?, C4 to C?, C5 to C?, C17 to C?, C3 to C?, C14 to C?, C15 to C?, C8 to C?, C12 to C?, C13 to C?, C2 to C?, C1 to C?, C9 to C?, C11 to C?, C7 to C?, C10 to C?, C16 to C?, D2 to D?, D1 to D?, F1 to F?, H1 to H?, H3 to H?, H2 to H?, H4 to H?, J1 to J?, J2 to J?, R3 to R?, R4 to R?, R5 to R?, R1 to R?, R2 to R?, SW1 to SW?, TP1 to TP?, TP5 to TP?, TP3 to TP?, TP4 to TP?, TP2 to TP?, U2 to U?, U3 to U?, U1 to U?, Y1 to Y?
Connections:
- net I2C2_SCL: now reaches U?.22 (PC4)
- net I2C2_SDA: now reaches U?.42 (PA8)
- no-connect marks 42 -> 40
