File: power-breadboard/nucleo64_stm32.kicad_sch (KiCad schematic)
At the start: 3 parts

Commit message: power-breadboard: complete nucleo peripheral table
Connections:
- net ~{DMS_PULSE_CLEAR} is gone; now on net DMS_FAULT_LATCH: J?.28 (Pin_28)
- net DMS_FAULT_LATCH: no longer J?.30 (Pin_30)
- net DMS_RESET: now also J?.30 (Pin_30); no longer J?.32 (Pin_32)
- net DMS_STATUS: now also J?.32 (Pin_32); no longer J?.34 (Pin_34)
- no-connect marks 43 -> 44

Commit message: power-breadboard: annotate whole schematic
Parts:
- gave numbers to parts that had none: 2
- renumbered R14 to R1
Changed lines of the file:
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@@
 		(dnp no)
 		(fields_autoplaced yes)
-		(property "Reference" "#PWR049"
+		(property "Reference" "#PWR013"
 			(at 33.02 50.8 0)
 			(hide yes)
@@
 			(project "power-breadboard"
 				(path "/4b4cf3aa-c94c-4150-b9c5-35049cd71136/7d59fd70-1fff-4c9c-ae77-583b08aef567"
-					(reference "#PWR049")
+					(reference "#PWR013")
 					(unit 1)
 				)
@@
 		(in_pos_files yes)
 		(dnp no)
-		(property "Reference" "R14"
+		(property "Reference" "R1"
 			(at 39.37 39.37 90)
 			(show_name no)
@@
 			(project "power-breadboard"
 				(path "/4b4cf3aa-c94c-4150-b9c5-35049cd71136/7d59fd70-1fff-4c9c-ae77-583b08aef567"
-					(reference "R14")
+					(reference "R1")
 					(unit 1)
 					(variant
@@
 		(dnp no)
 		(fields_autoplaced yes)
-		(property "Reference" "#PWR015"
+		(property "Reference" "#PWR011"
 			(at 45.72 26.67 0)
 			(hide yes)
@@
 			(project "power-breadboard"
 				(path "/4b4cf3aa-c94c-4150-b9c5-35049cd71136/7d59fd70-1fff-4c9c-ae77-583b08aef567"
-					(reference "#PWR015")
+					(reference "#PWR011")
 					(unit 1)
 				)
@@
 		(dnp no)
 		(fields_autoplaced yes)
-		(property "Reference" "J?"
+		(property "Reference" "J3"
 			(at 127 34.29 0)
 			(show_name no)
@@
 			(project "power-breadboard"
 				(path "/4b4cf3aa-c94c-4150-b9c5-35049cd71136/7d59fd70-1fff-4c9c-ae77-583b08aef567"
-					(reference "J?")
+					(reference "J3")
 					(unit 1)
 				)
@@
 		(dnp no)
 		(fields_autoplaced yes)
-		(property "Reference" "#PWR012"
+		(property "Reference" "#PWR015"
 			(at 66.04 92.71 0)
 			(hide yes)
@@
 			(project "power-breadboard"
 				(path "/4b4cf3aa-c94c-4150-b9c5-35049cd71136/7d59fd70-1fff-4c9c-ae77-583b08aef567"
-					(reference "#PWR012")
+					(reference "#PWR015")
 					(unit 1)
 				)
@@
 		(dnp no)
 		(fields_autoplaced yes)
-		(property "Reference" "J?"
+		(property "Reference" "J2"
 			(at 57.15 27.94 0)
 			(show_name no)
@@
 			(project "power-breadboard"
 				(path "/4b4cf3aa-c94c-4150-b9c5-35049cd71136/7d59fd70-1fff-4c9c-ae77-583b08aef567"
-					(reference "J?")
+					(reference "J2")
 					(unit 1)
 				)
@@
 		(dnp no)
 		(fields_autoplaced yes)
-		(property "Reference" "#PWR011"
+		(property "Reference" "#PWR012"
 			(at 68.58 26.67 0)
 			(hide yes)
@@
 			(project "power-breadboard"
 				(path "/4b4cf3aa-c94c-4150-b9c5-35049cd71136/7d59fd70-1fff-4c9c-ae77-583b08aef567"
-					(reference "#PWR011")
+					(reference "#PWR012")
 					(unit 1)
 				)
