File: power-breadboard/relay_board_connections.kicad_sch (KiCad schematic)
At the start: 11 parts

Commit message: power-pcb: add imd input to safety systems page
Use the same CAN transceiver as for the network since it also supports
24V-CAN. Also re-added a separate 24V input for the contactors.
Connections:
- removed net +24V: U?., U?., U?.
- new net: #OUT3. (GND), U?.
- new net: #OUT2. (GND), U?.
- new net: #OUT4. (GND), U?.
- new net: #OUT1. (GND), U?.
- new net: #OUT6. (GND), U?.
- new net: #OUT7. (GND), U?.
- new net: #OUT8. (GND), U?.
- new net: #OUT5. (GND), U?.
- new net CONTACTORS_24V: U?., U?., U?.
Other:
- title: Relay Board Connection -> Relay Board Connections
Changed lines of the file:
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@@
 	(paper "A4")
 	(title_block
-		(title "Relay Board Connection")
-		(date "2026-06-29")
+		(title "Relay Board Connections")
+		(date "2026-07-01")
 		(rev "v1.1.0")
 	)
@@
 	(wire
 		(pts
+			(xy 77.47 21.59) (xy 80.01 21.59)
+		)
+		(stroke
+			(width 0)
+			(type default)
+			(color 194 0 194 1)
+		)
+	)
+	(wire
+		(pts
 			(xy 64.77 121.92) (xy 59.69 121.92)
 		)
@@
 		)
 	)
+	(hierarchical_label "CONTACTORS_24V"
+		(shape input)
+		(at 77.47 21.59 180)
+		(effects
+			(font
+				(size 1.27 1.27)
+			)
+			(justify right)
+		)
+	)
 	(hierarchical_label "~{BRAKING_RESISTOR_SWITCH}"
 		(shape input)
@@
 			)
 			(justify right)
-		)
-	)
-	(symbol
-		(lib_id "power:+24V")
-		(at 80.01 21.59 0)
-		(unit 1)
-		(body_style 1)
-		(exclude_from_sim no)
-		(in_bom yes)
-		(on_board yes)
-		(in_pos_files yes)
-		(dnp no)
-		(fields_autoplaced yes)
-		(property "Reference" "#PWR04"
-			(at 80.01 25.4 0)
-			(hide yes)
-			(show_name no)
-			(do_not_autoplace no)
-			(effects
-				(font
-					(size 1.27 1.27)
-				)
-			)
-		)
-		(property "Value" "+24V"
-			(at 80.01 16.51 0)
-			(show_name no)
-			(do_not_autoplace no)
-			(effects
-				(font
-					(size 1.27 1.27)
-				)
-			)
-		)
-		(property "Footprint" ""
-			(at 80.01 21.59 0)
-			(hide yes)
-			(show_name no)
-			(do_not_autoplace no)
-			(effects
-				(font
-					(size 1.27 1.27)
-				)
-			)
-		)
-		(property "Datasheet" ""
-			(at 80.01 21.59 0)
-			(hide yes)
-			(show_name no)
-			(do_not_autoplace no)
-			(effects
-				(font
-					(size 1.27 1.27)
-				)
-			)
-		)
-		(property "Description" "Power symbol creates a global label with name \"+24V\""
-			(at 80.01 21.59 0)
-			(hide yes)
-			(show_name no)
-			(do_not_autoplace no)
-			(effects
-				(font
-					(size 1.27 1.27)
-				)
-			)
-		)
-		(pin "1"
-		)
-		(instances
-			(project "power-breadboard"
-				(path "/4b4cf3aa-c94c-4150-b9c5-35049cd71136/9838bcc9-e766-495a-ad52-0ec70b90713f"
-					(reference "#PWR04")
-					(unit 1)
-				)
-			)
 		)
 	)
@@
 		(property "Description" "4-Relay Board"
 			(at 74.93 26.67 0)
+			(show_name no)
+			(do_not_autoplace no)
+			(effects
+				(font
+					(size 1.27 1.27)
+				)
+			)
+		)
+		(property "DIST" ""
+			(at 74.93 45.72 0)
+			(hide yes)
+			(show_name no)
+			(do_not_autoplace no)
+			(effects
+				(font
+					(size 1.27 1.27)
+				)
+			)
+		)
+		(property "Part Name" ""
+			(at 74.93 45.72 0)
+			(hide yes)
 			(show_name no)
 			(do_not_autoplace no)
@@
 			)
 		)
+		(property "DIST" ""
+			(at 74.93 113.03 0)
+			(hide yes)
+			(show_name no)
+			(do_not_autoplace no)
+			(effects
+				(font
+					(size 1.27 1.27)
+				)
+			)
+		)
+		(property "Part Name" ""
+			(at 74.93 113.03 0)
+			(hide yes)
+			(show_name no)
+			(do_not_autoplace no)
+			(effects
+				(font
+					(size 1.27 1.27)
+				)
+			)
+		)
 		(pin ""
 		)
@@
 			(at 74.93 82.55 0)
 			(hide yes)
+			(show_name no)
+			(do_not_autoplace no)
+			(effects
+				(font
+					(size 1.27 1.27)
+				)
+			)
+		)
+		(property "DIST" ""
+			(at 74.93 82.55 0)
+			(hide yes)
+			(show_name no)
+			(do_not_autoplace no)
+			(effects
+				(font
+					(size 1.27 1.27)
+				)
+			)
+		)
+		(property "Part Name" ""
+			(at 74.93 82.55 0)
+			(hide yes)

Commit message: power-breadboard: annotate whole schematic
Parts:
- gave numbers to parts that had none: 3
Connections:
- new net: #OUT3. (GND), U3.
- new net: #OUT2. (GND), U3.
- new net: #OUT4. (GND), U3.
- new net: #OUT1. (GND), U3.
- new net: #OUT6. (GND), U4.
- new net: #OUT7. (GND), U5.
- new net: #OUT8. (GND), U5.
- new net: #OUT5. (GND), U4.
Changed lines of the file:
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@@
 		(in_pos_files yes)
 		(dnp no)
-		(property "Reference" "U?"
+		(property "Reference" "U3"
 			(at 74.93 24.13 0)
 			(show_name no)
@@
 			(project "power-breadboard"
 				(path "/4b4cf3aa-c94c-4150-b9c5-35049cd71136/9838bcc9-e766-495a-ad52-0ec70b90713f"
-					(reference "U?")
+					(reference "U3")
 					(unit 1)
 				)
@@
 		(in_pos_files yes)
 		(dnp no)
-		(property "Reference" "U?"
+		(property "Reference" "U5"
 			(at 74.93 97.79 0)
 			(show_name no)
@@
 			(project "power-breadboard"
 				(path "/4b4cf3aa-c94c-4150-b9c5-35049cd71136/9838bcc9-e766-495a-ad52-0ec70b90713f"
-					(reference "U?")
+					(reference "U5")
 					(unit 1)
 				)
@@
 		(in_pos_files yes)
 		(dnp no)
-		(property "Reference" "U?"
+		(property "Reference" "U4"
 			(at 74.93 67.31 0)
 			(show_name no)
@@
 			(project "power-breadboard"
 				(path "/4b4cf3aa-c94c-4150-b9c5-35049cd71136/9838bcc9-e766-495a-ad52-0ec70b90713f"
-					(reference "U?")
+					(reference "U4")
 					(unit 1)
 				)
@@
 		(dnp no)
 		(fields_autoplaced yes)
-		(property "Reference" "#PWR018"
+		(property "Reference" "#PWR016"
 			(at 53.34 46.99 0)
 			(hide yes)
@@
 			(project "power-breadboard"
 				(path "/4b4cf3aa-c94c-4150-b9c5-35049cd71136/9838bcc9-e766-495a-ad52-0ec70b90713f"
-					(reference "#PWR018")
+					(reference "#PWR016")
 					(unit 1)
 				)
@@
 		(dnp no)
 		(fields_autoplaced yes)
-		(property "Reference" "#PWR016"
+		(property "Reference" "#PWR019"
 			(at 88.9 135.89 0)
 			(hide yes)
@@
 			(project "power-breadboard"
 				(path "/4b4cf3aa-c94c-4150-b9c5-35049cd71136/9838bcc9-e766-495a-ad52-0ec70b90713f"
-					(reference "#PWR016")
+					(reference "#PWR019")
 					(unit 1)
 				)
@@
 		(dnp no)
 		(fields_autoplaced yes)
-		(property "Reference" "#PWR013"
+		(property "Reference" "#PWR018"
 			(at 62.23 135.89 0)
 			(hide yes)
@@
 			(project "power-breadboard"
 				(path "/4b4cf3aa-c94c-4150-b9c5-35049cd71136/9838bcc9-e766-495a-ad52-0ec70b90713f"
-					(reference "#PWR013")
+					(reference "#PWR018")
 					(unit 1)
 				)

Commit message: power-breadboard: remove series resistor on FC TX
Connections:
- new net: #OUT3. (GND), U3.
- new net: #OUT2. (GND), U3.
- new net: #OUT4. (GND), U3.
- new net: #OUT1. (GND), U3.
- new net: #OUT6. (GND), U4.
- new net: #OUT7. (GND), U5.
- new net: #OUT8. (GND), U5.
- new net: #OUT5. (GND), U4.
Changed lines of the file:
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@@
 		(title "Relay Board Connections")
 		(date "2026-07-01")
-		(rev "v1.1.0")
+		(rev "v1.1.1")
 	)
 	(rectangle
