File: power-breadboard/safety_systems.kicad_sch (KiCad schematic)
At the start: 78 parts, among them J14 Screw_Terminal_01x02, J15 Screw_Terminal_01x03, J16 Screw_Terminal_01x02, J17 Screw_Terminal_01x04, Q1 AO3400A, Q2 AO3400A, Q3 AO3400A, Q4 AO3400A, Q5 AO3400A, Q6 AO3400A, Q7 AO3400A, Q8 AO3400A, U28 MCP6002T, U29 SN74HC02N, U30 J107F1AS125VDC.36, U31 J107F1AS125VDC.36, U32 SN74AHC123AN

Commit message: power-pcb: add imd input to safety systems page
Use the same CAN transceiver as for the network since it also supports
24V-CAN. Also re-added a separate 24V input for the contactors.
Parts:
- removed C67, C69: 100n, Capacitor_SMD:C_0402_1005Metric_Pad0.74x0.62mm_HandSolder, symbol Device:C
- removed D13, D14: SMF5.0A, Diode_SMD:D_SOD-123F, symbol Device:D_Zener
- removed D15, D16: 1N4148, Diode_THT:D_DO-35_SOD27_P7.62mm_Horizontal, symbol Device:D
- removed D17: BZX79-C4V7, Diode_THT:D_DO-35_SOD27_P7.62mm_Horizontal, symbol Device:D_Zener
- removed F5: 10A, Exocet:Fuseholder_Littelfuse_Combined, symbol Device:Fuse
- removed J15: Screw_Terminal_01x03, Exocet:Wuerth_Term_Blk_3pos_Side_Entry_5mm, symbol Connector:Screw_Terminal_01x03
- removed J16: Screw_Terminal_01x02, Exocet:Wuerth_Term_Blk_2pos_Side_Entry_5mm, symbol Connector:Screw_Terminal_01x02
- removed J17: Screw_Terminal_01x04, Exocet:Wuerth_Term_Blk_4pos_Side_Entry_5mm, symbol Connector:Screw_Terminal_01x04
- removed Q7: AO3400A, Package_TO_SOT_SMD:SOT-23_Handsoldering, symbol Exocet:AO3400A
- removed R42, R46: 12k, Resistor_SMD:R_0402_1005Metric_Pad0.72x0.64mm_HandSolder, symbol Device:R
- removed R49: 3.6k, Resistor_SMD:R_0603_1608Metric_Pad0.98x0.95mm_HandSolder, symbol Device:R
- removed R52: 6.8k, Resistor_SMD:R_0603_1608Metric_Pad0.98x0.95mm_HandSolder, symbol Device:R
- removed R63: 1.2k, Resistor_SMD:R_0603_1608Metric_Pad0.98x0.95mm_HandSolder, symbol Device:R
- removed R64: 5.1k, Resistor_SMD:R_0402_1005Metric_Pad0.72x0.64mm_HandSolder, symbol Device:R
- removed TP76, TP78, TP80, TP81, TP83, TP84, TP85, TP86, TP87, TP88, TP89, TP90, TP94, TP96, TP97: Pad, TestPoint:TestPoint_Pad_D1.5mm, symbol Connector:TestPoint
- removed TP77, TP93: Hole, TestPoint:TestPoint_THTPad_D2.0mm_Drill1.0mm, symbol Connector:TestPoint
- removed TP79, TP82, TP91: White, TestPoint:TestPoint_Keystone_5005-5009_Compact, symbol Connector:TestPoint
- removed TP92: Yellow, TestPoint:TestPoint_Keystone_5005-5009_Compact, symbol Connector:TestPoint
- removed TP95: Green, TestPoint:TestPoint_Keystone_5005-5009_Compact, symbol Connector:TestPoint
- removed U28: MCP6002T, Package_SO:SOIC-8_3.9x4.9mm_P1.27mm, symbol Device:Opamp_Dual
- removed U30, U31: J107F1AS125VDC.36, Relay_THT:Relay_SPDT_Omron-G5LE-1, symbol Exocet:J107F1AS
- added C? (x2): 100n, symbol Device:C
- added C?: 100n, Capacitor_SMD:C_0402_1005Metric_Pad0.74x0.62mm_HandSolder, symbol Device:C
- added F?: 10A, Exocet:Fuseholder_Littelfuse_Combined, symbol Device:Fuse
- added J?: Screw_Terminal_01x02, Exocet:Wuerth_Term_Blk_2pos_Side_Entry_5mm, symbol Connector:Screw_Terminal_01x02
- added J?: (no value), symbol Connector_Generic:Conn_01x06
- added Q?: 2N7000, symbol Simulation_SPICE:NMOS
- added R? (x2): 10k, Resistor_SMD:R_0402_1005Metric_Pad0.72x0.64mm_HandSolder, symbol Device:R
- added R?: 120, Resistor_THT:R_Axial_DIN0309_L9.0mm_D3.2mm_P12.70mm_Horizontal, symbol Device:R
- added R?: 1.2k, Resistor_SMD:R_0603_1608Metric_Pad0.98x0.95mm_HandSolder, symbol Device:R
- added U?: TS0010D, symbol Exocet:TS0010D
- added U?: MCP2562, Package_DIP:DIP-8_W7.62mm, symbol Interface_CAN_LIN:MCP2562-E-P
- Q1, Q2, Q3, Q4, Q5, Q6, Q8: value AO3400A -> 2N7000; footprint Package_TO_SOT_SMD:SOT-23_Handsoldering -> (none); symbol Exocet:AO3400A -> Simulation_SPICE:NMOS; JLCPCB C20917 -> (none); MFR Alpha & Omega Semiconductor Inc. -> Diotec Semiconductor; MPN AO3400A -> 2N7000
- R43, R47, R51, R53, R54, R55, R56, R57, R58, R59, R60, R61, R62, R66, R67, R68: value 12k -> 10k
- R44, R48: value 3.6k -> 3.3k
- R45, R50: value 6.8k -> 6.2k
Connections:
- net +24V: now also J?.1 (Pin_1), U?.
- net +3.3V: now also C?.1, U?.5 (Vio)
- net +5V: now also C?.2, R?.1, R?.1, R?.1, U?., U?.3 (VDD)
- net DMS_FAULT_LATCH: now also Q4.1 (D); no longer Q4.3 (D)
- net GND: now also Q1.3 (S), Q2.3 (S), Q3.3 (S), Q4.3 (S), Q5.3 (S), Q6.3 (S), Q8.3 (S), C?.1, C?.2, C?.2, J?.2 (Pin_2), J?.4 (Pin_4), Q?.3 (S), U?., U?.2 (VSS), U?.8 (STBY); no longer Q1.2 (S), Q2.2 (S), Q3.2 (S), Q4.2 (S), Q5.2 (S), Q6.2 (S), Q8.2 (S)
- net IMD_CAN_RX: now also U?.4 (RXD)
- net IMD_CAN_TX: now also U?.1 (TXD)
- net ~{ALARM}: now also Q3.1 (D), Q8.1 (D), C?.1, J?.3 (Pin_3), Q?.2 (G), R?.2; no longer Q3.3 (D), Q8.3 (D)
- net at R51.2: now also Q1.2 (G); no longer Q1.1 (G)
- net at R59.2, U29.12: now also Q6.1 (D); no longer Q6.3 (D)
- net at R57.2: now also Q2.2 (G); no longer Q2.1 (G)
- net at Q5.1 (D): now also R?.2, U?.; no longer R61.2
- net at R56.2: now also Q4.2 (G); no longer Q4.1 (G)
- net at R54.2, U29.8: now also Q2.1 (D); no longer Q2.3 (D)
- net at R67.2: now also Q8.2 (G); no longer Q8.1 (G)
- net at R62.2: now also Q6.2 (G); no longer Q6.1 (G)
- net at R58.2: now also Q3.2 (G); no longer Q3.1 (G)
- net at R43.2, U29.3: now also Q1.1 (D); no longer Q1.3 (D)
- new net: Q?.1 (D), R?.2, U?.
- new net: F?.1, U?.
- new net: J?.2 (Pin_2), U?.
- new net: Q5.2 (G), R61.2
- new net: J?.5 (Pin_5), R?.1, U?.7 (CANH)
- new net: J?.6 (Pin_6), R?.2, U?.6 (CANL)
- new net: F?.2, J?.1 (Pin_1)
- new net CONTACTORS_24V: U?.
- no-connect marks 4 -> 9
Other:
- removed sheet IMD Input
- note added: "Insulation Monitoring Device"
- note added: "Relay Ouptut Signals"
- note added: "Safety Relays"
- note removed: "Contactor Supply Relay"
- note removed: "Motor Key Relay"
- note removed: "Motor Throttle Input"
- moved on the sheet: C66, C68, J14, R43, R44, R45, R47, R48, R50, R51, R53, R54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

Commit message: power-breadboard: complete nucleo peripheral table
Connections:
- net ~{DMS_PULSE_CLEAR}: no longer names the net of R68.1, U32.3 (Clr)
Changed lines of the file:
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@@
-	)
-	(junction
-		(at 55.88 167.64)
-		(diameter 0)
-		(color 0 0 0 0)
 	)
 	(junction
@@
 		(pts
 			(xy 158.75 105.41) (xy 167.64 105.41)
-		)
-		(stroke
-			(width 0)
-			(type default)
-		)
-	)
-	(wire
-		(pts
-			(xy 41.91 167.64) (xy 55.88 167.64)
 		)
 		(stroke
@@
 		)
 	)
-	(hierarchical_label "~{DMS_PULSE_CLEAR}"
-		(shape input)
-		(at 41.91 167.64 180)
-		(effects
-			(font
-				(size 1.27 1.27)
-			)
-			(justify right)
-		)
-	)

Commit message: power-breadboard: annotate whole schematic
Parts:
- gave numbers to parts that had none: 13
- renumbered C68 to C10, C70 to C12, C71 to C13, C66 to C8, J14 to J6, Q3 to Q4, Q4 to Q5, Q5 to Q7, R43 to R18, R44 to R19, R45 to R20, R47 to R21, R48 to R22, R51 to R24, R50 to R25, R53 to R26, R54 to R27, R55 to R28, R56 to R31, R57 to R32, R58 to R33, R59 to R34, R60 to R36, R62 to R37, R61 to R38, R65 to R39, R66 to R40, R67 to R41, R68 to R42, U29 to U13, U32 to U16
